Commit message: Robot upgrades

File: src/maze_generator/urdf/mouse_full.xacro (robot description, xacro)
@@ -220,9 +220,9 @@
     <parent link="link_chassis"/>
     <child link="link_scan"/>
-    <origin xyz="0.02 0 0.05" rpy="0 0 0"/>
+    <origin xyz="0.15 0 0.06" rpy="0 0 -1.57079"/>
   </joint>
   <link name="link_scan">
     <visual>
-      <origin xyz="0 0 0.05" rpy="0 0 0"/>
+      <origin xyz="0 0 0" rpy="0 0 0"/>
       <geometry>
         <box size="0.05 0.05 0.05"/>
@@ -231,5 +231,5 @@
     </visual>
     <collision>
-      <origin xyz="0 0 0.05" rpy="0 0 0"/>
+      <origin xyz="0 0 0" rpy="0 0 0"/>
       <geometry>
         <box size="0.05 0.05 0.05"/>
@@ -253,5 +253,5 @@
             <resolution>1</resolution>
             <min_angle>0.0</min_angle>
-            <max_angle>6.28319</max_angle>
+            <max_angle>3.14159</max_angle>
           </horizontal>
         </scan>
