Commit message: Control implemented

File: src/maze_generator/urdf/mouse_lidar.xacro (robot description, xacro)
@@ -51,4 +51,16 @@
       <material name="blue"/>
     </visual>
+  </link>
+  <joint name="fixed_base_joint" type="fixed">
+    <origin rpy="0 0 0" xyz="0 0 0"/>
+    <child link="chassis_inertia"/>
+    <parent link="link_chassis"/>
+  </joint>
+  <link name="chassis_inertia">
+    <inertial>
+      <mass value="0.5"/>
+      <origin rpy="1.5707 0 1.5707" xyz="0 0 0"/>
+      <inertia ixx="0.0001062083333" ixy="0" ixz="0" iyy="0.0001416666667" iyz="0" izz="0.00003954166667"/>
+    </inertial>
   </link>
   <joint name="fixed_caster_joint" type="fixed">
@@ -81,21 +93,9 @@
     </visual>
   </link>
-  <joint name="fixed_base_joint" type="fixed">
-    <origin rpy="0 0 0" xyz="0 0 0"/>
-    <child link="chassis_inertia"/>
-    <parent link="link_chassis"/>
-  </joint>
-  <link name="chassis_inertia">
-    <inertial>
-      <mass value="0.5"/>
-      <origin rpy="1.5707 0 1.5707" xyz="0 0 0"/>
-      <inertia ixx="0.0001062083333" ixy="0" ixz="0" iyy="0.0001416666667" iyz="0" izz="0.00003954166667"/>
-    </inertial>
-  </link>
   <link name="link_right_wheel">
     <inertial>
       <mass value="0.02"/>
       <origin rpy="0 1.5707 1.5707" xyz="0 0 0"/>
-      <inertia ixx="0.000000526666666667" ixy="0" ixz="0" iyy="0.000000526666666667" iyz="0" izz="0.00000016"/>
+      <inertia ixx="5.267e-7" ixy="0" ixz="0" iyy="5.267e-7" iyz="0" izz="1e-6"/>
     </inertial>
     <collision name="link_right_wheel_collision">
@@ -124,5 +124,5 @@
       <mass value="0.02"/>
       <origin rpy="0 1.5707 1.5707" xyz="0 0 0"/>
-      <inertia ixx="0.000000526666666667" ixy="0" ixz="0" iyy="0.000000526666666667" iyz="0" izz="0.00000016"/>
+      <inertia ixx="5.267e-7" ixy="0" ixz="0" iyy="5.267e-7" iyz="0" izz="1e-6"/>
     </inertial>
     <collision name="link_left_wheel_collision">
@@ -147,31 +147,4 @@
     <joint_properties damping="1.0" friction="1.0"/>
   </joint>
-  <!-- Simulation behavior -->
-  <gazebo reference="link_left_wheel">
-    <mu1>0.1</mu1>
-    <mu2>0.1</mu2>
-    <kp>500000.0</kp>
-    <kd>10.0</kd>
-    <minDepth>0.001</minDepth>
-    <maxVel>0.1</maxVel>
-    <fdir1>1 0 0</fdir1>
-  </gazebo>
-  <gazebo reference="link_right_wheel">
-    <mu1>0.1</mu1>
-    <mu2>0.1</mu2>
-    <kp>500000.0</kp>
-    <kd>10.0</kd>
-    <minDepth>0.001</minDepth>
-    <maxVel>0.1</maxVel>
-    <fdir1>1 0 0</fdir1>
-  </gazebo>
-  <gazebo reference="link_chassis">
-    <mu1>0.1</mu1>
-    <mu2>0.1</mu2>
-    <kp>1000000.0</kp>
-    <kd>100.0</kd>
-    <minDepth>0.001</minDepth>
-    <maxVel>1.0</maxVel>
-  </gazebo>
   <!-- IMU Sensor -->
   <link name="imu_link"/>
@@ -290,6 +263,6 @@
       <leftJoint>joint_left_wheel</leftJoint>
       <rightJoint>joint_right_wheel</rightJoint>
-      <wheelSeparation>0.287</wheelSeparation>
-      <wheelDiameter>0.066</wheelDiameter>
+      <wheelSeparation>0.03</wheelSeparation>
+      <wheelDiameter>0.02</wheelDiameter>
       <wheelAcceleration>1</wheelAcceleration>
       <wheelTorque>10</wheelTorque>

Commit message: Fixed inertias

File: src/maze_generator/urdf/mouse_lidar.xacro (robot description, xacro)
@@ -60,6 +60,6 @@
     <inertial>
       <mass value="0.5"/>
-      <origin rpy="1.5707 0 1.5707" xyz="0 0 0"/>
-      <inertia ixx="0.0001062083333" ixy="0" ixz="0" iyy="0.0001416666667" iyz="0" izz="0.00003954166667"/>
+      <origin rpy="0 0 0" xyz="0 0 0"/>
+      <inertia ixx="0.00003954166667" ixy="0" ixz="0" iyy="0.0001062083333" iyz="0" izz="0.0001416666667"/>
     </inertial>
   </link>
@@ -209,9 +209,4 @@
       </geometry>
     </collision>
-    <inertial>
-      <mass value="0.01" />
-      <origin xyz="0 0 0" />
-      <inertia ixx="0.0001" ixy="0.0" ixz="0.0" iyy="0.0001" iyz="0.0" izz="0.0001" />
-    </inertial>
   </link>
   <gazebo reference="link_scan">
