Commit message: Robot model

File: src/maze_generator/urdf/mouse.xacro (robot description, xacro)
@@ -1,4 +1,4 @@
 <?xml version="1.0" ?>
-<robot name="m2wr" xmlns:xacro="http://www.ros.org/wiki/xacro">
+<robot name="mouse" xmlns:xacro="http://www.ros.org/wiki/xacro">
   <material name="black">
     <color rgba="0.0 0.0 0.0 1.0"/>
@@ -51,11 +51,6 @@
   </gazebo>
   <link name="link_chassis">
-    <!-- pose and inertial -->
+    <!-- pose -->
     <pose>0 0 0.1 0 0 0</pose>
-    <inertial>
-      <mass value="5"/>
-      <origin rpy="0 0 0" xyz="0 0 0.1"/>
-      <inertia ixx="0.0395416666667" ixy="0" ixz="0" iyy="0.106208333333" iyz="0" izz="0.106208333333"/>
-    </inertial>
     <!-- body -->
     <collision name="collision_chassis">
@@ -94,4 +89,16 @@
       </geometry>
     </visual>
+  </link>
+  <joint name="fixed_base_joint" type="fixed">
+    <origin rpy="0 0 0" xyz="0 0 0"/>
+    <child link="chassis_inertia"/>
+    <parent link="link_chassis"/>
+  </joint>
+  <link name="chassis_inertia">
+    <inertial>
+      <mass value="5"/>
+      <origin rpy="0 0 0" xyz="0 0 0.1"/>
+      <inertia ixx="0.0395416666667" ixy="0" ixz="0" iyy="0.106208333333" iyz="0" izz="0.106208333333"/>
+    </inertial>
   </link>
   <link name="link_right_wheel">

Commit message: IR sensor added

File: src/maze_generator/urdf/mouse.xacro (robot description, xacro)
@@ -156,3 +156,59 @@
     <joint_properties damping="1.0" friction="1.0"/>
   </joint>
+  <joint name="fixed_sensor" type="fixed">
+    <origin rpy="0 0 0" xyz="0 0 0"/>
+    <child link="link_infrared"/>
+    <parent link="link_chassis"/>
+  </joint>
+  <link name="link_infrared">
+    <collision>
+      <origin rpy="0 0 0" xyz="0.25 0 0"/>
+      <geometry>
+        <box size="0.05 0.05 0.05"/>
+      </geometry>
+    </collision>
+    <visual>
+      <origin rpy="0 0 0" xyz="0.25 0 0"/>
+      <geometry>
+        <box size="0.05 0.05 0.05"/>
+      </geometry>
+    </visual>
+  </link>
+  <gazebo reference="link_chassis">
+   <sensor type="ray" name="TeraRanger">
+      <pose>0.275 0 0 0 0 0</pose>
+      <visualize>true</visualize>
+      <update_rate>50</update_rate>
+      <ray>
+         <scan>
+            <horizontal>
+               <samples>10</samples>
+               <resolution>1</resolution>
+               <min_angle>-0.14835</min_angle>
+               <max_angle>0.14835</max_angle>
+            </horizontal>
+            <vertical>
+               <samples>10</samples>
+               <resolution>1</resolution>
+               <min_angle>-0.14835</min_angle>
+               <max_angle>0.14835</max_angle>
+            </vertical>
+         </scan>
+         <range>
+            <min>0.01</min>
+            <max>2</max>
+            <resolution>0.02</resolution>
+         </range>
+      </ray>
+      <plugin filename="libgazebo_ros_range.so" name="gazebo_ros_range">
+         <gaussianNoise>0.005</gaussianNoise>
+         <alwaysOn>true</alwaysOn>
+         <updateRate>50</updateRate>
+         <topicName>sensor/infrared</topicName>
+         <frameName>link_infrared</frameName>
+         <radiation>INFRARED</radiation>
+         <fov>0.2967</fov>
+      </plugin>
+   </sensor>
+   </gazebo>
 </robot>

Commit message: fix range rviz

File: src/maze_generator/urdf/mouse.xacro (robot description, xacro)
@@ -157,5 +157,5 @@
   </joint>
   <joint name="fixed_sensor" type="fixed">
-    <origin rpy="0 0 0" xyz="0 0 0"/>
+    <origin rpy="0 0 0" xyz="0.275 0 0"/>
     <child link="link_infrared"/>
     <parent link="link_chassis"/>
@@ -163,5 +163,5 @@
   <link name="link_infrared">
     <collision>
-      <origin rpy="0 0 0" xyz="0.25 0 0"/>
+      <origin rpy="0 0 0" xyz="0 0 0"/>
       <geometry>
         <box size="0.05 0.05 0.05"/>
@@ -169,5 +169,5 @@
     </collision>
     <visual>
-      <origin rpy="0 0 0" xyz="0.25 0 0"/>
+      <origin rpy="0 0 0" xyz="0 0 0"/>
       <geometry>
         <box size="0.05 0.05 0.05"/>
@@ -177,5 +177,5 @@
   <gazebo reference="link_chassis">
    <sensor type="ray" name="TeraRanger">
-      <pose>0.275 0 0 0 0 0</pose>
+      <pose>0 0 0 0 0 0</pose>
       <visualize>true</visualize>
       <update_rate>50</update_rate>

Commit message: Working sensor

File: src/maze_generator/urdf/mouse.xacro (robot description, xacro)
@@ -68,5 +68,5 @@
     <!-- caster front -->
     <collision name="caster_front_collision">
-      <origin rpy=" 0 0 0" xyz="0.35 0 -0.05"/>
+      <origin rpy="0 0 0" xyz="0.2 0 -0.05"/>
       <geometry>
         <sphere radius="0.05"/>
@@ -84,5 +84,5 @@
     </collision>
     <visual name="caster_front_visual">
-      <origin rpy=" 0 0 0" xyz="0.2 0 -0.05"/>
+      <origin rpy="0 0 0" xyz="0.2 0 -0.05"/>
       <geometry>
         <sphere radius="0.05"/>
@@ -162,10 +162,4 @@
   </joint>
   <link name="link_infrared">
-    <collision>
-      <origin rpy="0 0 0" xyz="0 0 0"/>
-      <geometry>
-        <box size="0.05 0.05 0.05"/>
-      </geometry>
-    </collision>
     <visual>
       <origin rpy="0 0 0" xyz="0 0 0"/>
@@ -175,5 +169,5 @@
     </visual>
   </link>
-  <gazebo reference="link_chassis">
+  <gazebo reference="link_infrared">
    <sensor type="ray" name="TeraRanger">
       <pose>0 0 0 0 0 0</pose>

Commit message: resize mouse

File: src/maze_generator/urdf/mouse.xacro (robot description, xacro)
@@ -56,5 +56,5 @@
     <collision name="collision_chassis">
       <geometry>
-        <box size="0.5 0.3 0.07"/>
+        <box size="0.05 0.03 0.007"/>
       </geometry>
     </collision>
@@ -62,5 +62,5 @@
       <origin rpy="0 0 0" xyz="0 0 0"/>
       <geometry>
-        <box size="0.5 0.3 0.07"/>
+        <box size="0.05 0.03 0.007"/>
       </geometry>
       <material name="blue"/>
@@ -68,7 +68,7 @@
     <!-- caster front -->
     <collision name="caster_front_collision">
-      <origin rpy="0 0 0" xyz="0.2 0 -0.05"/>
-      <geometry>
-        <sphere radius="0.05"/>
+      <origin rpy="0 0 0" xyz="0.018 0 -0.005"/>
+      <geometry>
+        <sphere radius="0.006"/>
       </geometry>
       <surface>
@@ -84,7 +84,7 @@
     </collision>
     <visual name="caster_front_visual">
-      <origin rpy="0 0 0" xyz="0.2 0 -0.05"/>
-      <geometry>
-        <sphere radius="0.05"/>
+      <origin rpy="0 0 0" xyz="0.018 0 -0.005"/>
+      <geometry>
+        <sphere radius="0.006"/>
       </geometry>
     </visual>
@@ -111,5 +111,5 @@
       <origin rpy="0 1.5707 1.5707" xyz="0 0 0"/>
       <geometry>
-        <cylinder length="0.04" radius="0.1"/>
+        <cylinder length="0.004" radius="0.01"/>
       </geometry>
     </collision>
@@ -117,10 +117,10 @@
       <origin rpy="0 1.5707 1.5707" xyz="0 0 0"/>
       <geometry>
-        <cylinder length="0.04" radius="0.1"/>
+        <cylinder length="0.004" radius="0.01"/>
       </geometry>
     </visual>
   </link>
   <joint name="joint_right_wheel" type="continuous">
-    <origin rpy="0 0 0" xyz="-0.05 0.15 0"/>
+    <origin rpy="0 0 0" xyz="-0.005 0.015 0"/>
     <child link="link_right_wheel"/>
     <parent link="link_chassis"/>
@@ -138,5 +138,5 @@
       <origin rpy="0 1.5707 1.5707" xyz="0 0 0"/>
       <geometry>
-        <cylinder length="0.04" radius="0.1"/>
+        <cylinder length="0.004" radius="0.01"/>
       </geometry>
     </collision>
@@ -144,10 +144,10 @@
       <origin rpy="0 1.5707 1.5707" xyz="0 0 0"/>
       <geometry>
-        <cylinder length="0.04" radius="0.1"/>
+        <cylinder length="0.004" radius="0.01"/>
       </geometry>
     </visual>
   </link>
   <joint name="joint_left_wheel" type="continuous">
-    <origin rpy="0 0 0" xyz="-0.05 -0.15 0"/>
+    <origin rpy="0 0 0" xyz="-0.005 -0.015 0"/>
     <child link="link_left_wheel"/>
     <parent link="link_chassis"/>
@@ -157,5 +157,5 @@
   </joint>
   <joint name="fixed_sensor" type="fixed">
-    <origin rpy="0 0 0" xyz="0.275 0 0"/>
+    <origin rpy="0 0 0" xyz="0.0275 0 0"/>
     <child link="link_infrared"/>
     <parent link="link_chassis"/>
@@ -165,5 +165,5 @@
       <origin rpy="0 0 0" xyz="0 0 0"/>
       <geometry>
-        <box size="0.05 0.05 0.05"/>
+        <box size="0.005 0.005 0.005"/>
       </geometry>
     </visual>

Commit message: resize 2

File: src/maze_generator/urdf/mouse.xacro (robot description, xacro)
@@ -68,7 +68,7 @@
     <!-- caster front -->
     <collision name="caster_front_collision">
-      <origin rpy="0 0 0" xyz="0.018 0 -0.005"/>
-      <geometry>
-        <sphere radius="0.006"/>
+      <origin rpy="0 0 0" xyz="0.02 0 -0.005"/>
+      <geometry>
+        <sphere radius="0.005"/>
       </geometry>
       <surface>
@@ -86,5 +86,5 @@
       <origin rpy="0 0 0" xyz="0.018 0 -0.005"/>
       <geometry>
-        <sphere radius="0.006"/>
+        <sphere radius="0.005"/>
       </geometry>
     </visual>
@@ -97,5 +97,5 @@
   <link name="chassis_inertia">
     <inertial>
-      <mass value="5"/>
+      <mass value="0.5"/>
       <origin rpy="0 0 0" xyz="0 0 0.1"/>
       <inertia ixx="0.0395416666667" ixy="0" ixz="0" iyy="0.106208333333" iyz="0" izz="0.106208333333"/>
@@ -104,5 +104,5 @@
   <link name="link_right_wheel">
     <inertial>
-      <mass value="0.2"/>
+      <mass value="0.02"/>
       <origin rpy="0 1.5707 1.5707" xyz="0 0 0"/>
       <inertia ixx="0.000526666666667" ixy="0" ixz="0" iyy="0.000526666666667" iyz="0" izz="0.001"/>
@@ -131,5 +131,5 @@
   <link name="link_left_wheel">
     <inertial>
-      <mass value="0.2"/>
+      <mass value="0.02"/>
       <origin rpy="0 1.5707 1.5707" xyz="0 0 0"/>
       <inertia ixx="0.000526666666667" ixy="0" ixz="0" iyy="0.000526666666667" iyz="0" izz="0.001"/>

Commit message: Inertias

File: src/maze_generator/urdf/mouse.xacro (robot description, xacro)
@@ -98,6 +98,6 @@
     <inertial>
       <mass value="0.5"/>
-      <origin rpy="0 0 0" xyz="0 0 0.1"/>
-      <inertia ixx="0.0395416666667" ixy="0" ixz="0" iyy="0.106208333333" iyz="0" izz="0.106208333333"/>
+      <origin rpy="1.5707 0 1.5707" xyz="0 0 0"/>
+      <inertia ixx="0.0001062083333" ixy="0" ixz="0" iyy="0.0001416666667" iyz="0" izz="0.00003954166667"/>
     </inertial>
   </link>
@@ -106,5 +106,5 @@
       <mass value="0.02"/>
       <origin rpy="0 1.5707 1.5707" xyz="0 0 0"/>
-      <inertia ixx="0.000526666666667" ixy="0" ixz="0" iyy="0.000526666666667" iyz="0" izz="0.001"/>
+      <inertia ixx="0.000000526666666667" ixy="0" ixz="0" iyy="0.000000526666666667" iyz="0" izz="0.00000016"/>
     </inertial>
     <collision name="link_right_wheel_collision">
@@ -133,5 +133,5 @@
       <mass value="0.02"/>
       <origin rpy="0 1.5707 1.5707" xyz="0 0 0"/>
-      <inertia ixx="0.000526666666667" ixy="0" ixz="0" iyy="0.000526666666667" iyz="0" izz="0.001"/>
+      <inertia ixx="0.000000526666666667" ixy="0" ixz="0" iyy="0.000000526666666667" iyz="0" izz="0.00000016"/>
     </inertial>
     <collision name="link_left_wheel_collision">

Commit message: fix ball collision

File: src/maze_generator/urdf/mouse.xacro (robot description, xacro)
@@ -84,5 +84,5 @@
     </collision>
     <visual name="caster_front_visual">
-      <origin rpy="0 0 0" xyz="0.018 0 -0.005"/>
+      <origin rpy="0 0 0" xyz="0.02 0 -0.005"/>
       <geometry>
         <sphere radius="0.005"/>
