Commit message: Robot models finished

File: src/maze_generator/urdf/mouse_lidar.xacro (robot description, xacro)
@@ -28,4 +28,7 @@
     <material>Gazebo/Orange</material>
   </gazebo>
+  <gazebo reference="link_caster">
+    <material>Gazebo/Gray</material>
+  </gazebo>
   <gazebo reference="link_left_wheel">
     <material>Gazebo/Blue</material>
@@ -34,27 +37,9 @@
     <material>Gazebo/Blue</material>
   </gazebo>
-  <gazebo>
-    <plugin filename="libgazebo_ros_diff_drive.so" name="differential_drive_controller">
-      <legacyMode>false</legacyMode>
-      <alwaysOn>true</alwaysOn>
-      <updateRate>20</updateRate>
-      <leftJoint>joint_left_wheel</leftJoint>
-      <rightJoint>joint_right_wheel</rightJoint>
-      <wheelSeparation>0.2</wheelSeparation>
-      <wheelDiameter>0.2</wheelDiameter>
-      <torque>0.1</torque>
-      <commandTopic>cmd_vel</commandTopic>
-      <odometryTopic>odom</odometryTopic>
-      <odometryFrame>odom</odometryFrame>
-      <robotBaseFrame>link_chassis</robotBaseFrame>
-    </plugin>
-  </gazebo>
+  <!-- Robot description -->
   <link name="link_chassis">
-    <!-- pose -->
-    <pose>0 0 0.1 0 0 0</pose>
-    <!-- body -->
     <collision name="collision_chassis">
       <geometry>
-        <box size="0.5 0.3 0.07"/>
+        <box size="0.05 0.03 0.007"/>
       </geometry>
     </collision>
@@ -62,13 +47,19 @@
       <origin rpy="0 0 0" xyz="0 0 0"/>
       <geometry>
-        <box size="0.5 0.3 0.07"/>
+        <box size="0.05 0.03 0.007"/>
       </geometry>
       <material name="blue"/>
     </visual>
-    <!-- caster front -->
+  </link>
+  <joint name="fixed_caster_joint" type="fixed">
+    <origin rpy="0 0 0" xyz="0 0 0"/>
+    <child link="link_caster"/>
+    <parent link="link_chassis"/>
+  </joint>
+  <link name="link_caster">
     <collision name="caster_front_collision">
-      <origin rpy="0 0 0" xyz="0.2 0 -0.05"/>
-      <geometry>
-        <sphere radius="0.05"/>
+      <origin rpy="0 0 0" xyz="0.02 0 -0.005"/>
+      <geometry>
+        <sphere radius="0.005"/>
       </geometry>
       <surface>
@@ -84,7 +75,7 @@
     </collision>
     <visual name="caster_front_visual">
-      <origin rpy="0 0 0" xyz="0.2 0 -0.05"/>
-      <geometry>
-        <sphere radius="0.05"/>
+      <origin rpy="0 0 0" xyz="0.02 0 -0.005"/>
+      <geometry>
+        <sphere radius="0.005"/>
       </geometry>
     </visual>
@@ -97,19 +88,19 @@
   <link name="chassis_inertia">
     <inertial>
-      <mass value="5"/>
-      <origin rpy="0 0 0" xyz="0 0 0.1"/>
-      <inertia ixx="0.0395416666667" ixy="0" ixz="0" iyy="0.106208333333" iyz="0" izz="0.106208333333"/>
+      <mass value="0.5"/>
+      <origin rpy="1.5707 0 1.5707" xyz="0 0 0"/>
+      <inertia ixx="0.0001062083333" ixy="0" ixz="0" iyy="0.0001416666667" iyz="0" izz="0.00003954166667"/>
     </inertial>
   </link>
   <link name="link_right_wheel">
     <inertial>
-      <mass value="0.2"/>
-      <origin rpy="0 1.5707 1.5707" xyz="0 0 0"/>
-      <inertia ixx="0.000526666666667" ixy="0" ixz="0" iyy="0.000526666666667" iyz="0" izz="0.001"/>
+      <mass value="0.02"/>
+      <origin rpy="0 1.5707 1.5707" xyz="0 0 0"/>
+      <inertia ixx="0.000000526666666667" ixy="0" ixz="0" iyy="0.000000526666666667" iyz="0" izz="0.00000016"/>
     </inertial>
     <collision name="link_right_wheel_collision">
       <origin rpy="0 1.5707 1.5707" xyz="0 0 0"/>
       <geometry>
-        <cylinder length="0.04" radius="0.1"/>
+        <cylinder length="0.004" radius="0.01"/>
       </geometry>
     </collision>
@@ -117,10 +108,10 @@
       <origin rpy="0 1.5707 1.5707" xyz="0 0 0"/>
       <geometry>
-        <cylinder length="0.04" radius="0.1"/>
+        <cylinder length="0.004" radius="0.01"/>
       </geometry>
     </visual>
   </link>
   <joint name="joint_right_wheel" type="continuous">
-    <origin rpy="0 0 0" xyz="-0.05 0.15 0"/>
+    <origin rpy="0 0 0" xyz="-0.005 0.015 0"/>
     <child link="link_right_wheel"/>
     <parent link="link_chassis"/>
@@ -131,12 +122,12 @@
   <link name="link_left_wheel">
     <inertial>
-      <mass value="0.2"/>
-      <origin rpy="0 1.5707 1.5707" xyz="0 0 0"/>
-      <inertia ixx="0.000526666666667" ixy="0" ixz="0" iyy="0.000526666666667" iyz="0" izz="0.001"/>
+      <mass value="0.02"/>
+      <origin rpy="0 1.5707 1.5707" xyz="0 0 0"/>
+      <inertia ixx="0.000000526666666667" ixy="0" ixz="0" iyy="0.000000526666666667" iyz="0" izz="0.00000016"/>
     </inertial>
     <collision name="link_left_wheel_collision">
       <origin rpy="0 1.5707 1.5707" xyz="0 0 0"/>
       <geometry>
-        <cylinder length="0.04" radius="0.1"/>
+        <cylinder length="0.004" radius="0.01"/>
       </geometry>
     </collision>
@@ -144,10 +135,10 @@
       <origin rpy="0 1.5707 1.5707" xyz="0 0 0"/>
       <geometry>
-        <cylinder length="0.04" radius="0.1"/>
+        <cylinder length="0.004" radius="0.01"/>
       </geometry>
     </visual>
   </link>
   <joint name="joint_left_wheel" type="continuous">
-    <origin rpy="0 0 0" xyz="-0.05 -0.15 0"/>
+    <origin rpy="0 0 0" xyz="-0.005 -0.015 0"/>
     <child link="link_left_wheel"/>
     <parent link="link_chassis"/>
@@ -156,53 +147,153 @@
     <joint_properties damping="1.0" friction="1.0"/>
   </joint>
-  <joint name="fixed_sensor" type="fixed">
-    <origin rpy="0 0 0" xyz="0.275 0 0"/>
-    <child link="link_infrared"/>
-    <parent link="link_chassis"/>
-  </joint>
-  <link name="link_infrared">
+  <!-- Simulation behavior -->
+  <gazebo reference="link_left_wheel">
+    <mu1>0.1</mu1>
+    <mu2>0.1</mu2>
+    <kp>500000.0</kp>
+    <kd>10.0</kd>
+    <minDepth>0.001</minDepth>
+    <maxVel>0.1</maxVel>
+    <fdir1>1 0 0</fdir1>
+  </gazebo>
+  <gazebo reference="link_right_wheel">
+    <mu1>0.1</mu1>
+    <mu2>0.1</mu2>
+    <kp>500000.0</kp>
+    <kd>10.0</kd>
+    <minDepth>0.001</minDepth>
+    <maxVel>0.1</maxVel>
+    <fdir1>1 0 0</fdir1>
+  </gazebo>
+  <gazebo reference="link_chassis">
+    <mu1>0.1</mu1>
+    <mu2>0.1</mu2>
+    <kp>1000000.0</kp>
+    <kd>100.0</kd>
+    <minDepth>0.001</minDepth>
+    <maxVel>1.0</maxVel>
+  </gazebo>
+  <!-- IMU Sensor -->
+  <link name="imu_link"/>
+  <joint name="imu_joint" type="fixed">
+    <parent link="link_chassis"/>
+    <child link="imu_link"/>
+    <origin xyz="0 0 0" rpy="0 0 0"/>
+  </joint>
+  <gazebo reference="imu_link">
+    <sensor type="imu" name="imu">
+      <always_on>true</always_on>
+      <visualize>true</visualize>
+    </sensor>
+    <material>Gazebo/Grey</material>
+  </gazebo>
+  <gazebo>
+    <plugin name="imu_plugin" filename="libgazebo_ros_imu.so">
+      <alwaysOn>true</alwaysOn>
+      <bodyName>imu_link</bodyName>
+      <frameName>imu_link</frameName>
+      <topicName>imu</topicName>
+      <serviceName>imu_service</serviceName>
+      <gaussianNoise>0.0</gaussianNoise>
+      <updateRate>200</updateRate>
+      <imu>
+        <noise>
+          <type>gaussian</type>
+          <rate>
+            <mean>0.0</mean>
+            <stddev>2e-4</stddev>
+            <bias_mean>0.0000075</bias_mean>
+            <bias_stddev>0.0000008</bias_stddev>
+          </rate>
+          <accel>
+            <mean>0.0</mean>
+            <stddev>1.7e-2</stddev>
+            <bias_mean>0.1</bias_mean>
+            <bias_stddev>0.001</bias_stddev>
+          </accel>
+        </noise>
+      </imu>
+    </plugin>
+  </gazebo>
+  <!-- LiDAR Sensor -->
+  <joint name="scan_joint" type="fixed">
+    <parent link="link_chassis"/>
+    <child link="link_scan"/>
+    <origin xyz="0.015 0 0.006" rpy="0 0 -1.57079"/>
+  </joint>
+  <link name="link_scan">
     <visual>
-      <origin rpy="0 0 0" xyz="0 0 0"/>
-      <geometry>
-        <box size="0.05 0.05 0.05"/>
-      </geometry>
-    </visual>
-  </link>
-  <gazebo reference="link_infrared">
-   <sensor type="ray" name="TeraRanger">
+      <origin xyz="0 0 0" rpy="0 0 0"/>
+      <geometry>
+        <box size="0.005 0.005 0.005"/>
+      </geometry>
+      <material name="black"/>
+    </visual>
+    <collision>
+      <origin xyz="0 0 0" rpy="0 0 0"/>
+      <geometry>
+        <box size="0.005 0.005 0.005"/>
+      </geometry>
+    </collision>
+    <inertial>
+      <mass value="0.01" />
+      <origin xyz="0 0 0" />
+      <inertia ixx="0.0001" ixy="0.0" ixz="0.0" iyy="0.0001" iyz="0.0" izz="0.0001" />
+    </inertial>
+  </link>
+  <gazebo reference="link_scan">
+    <sensor type="ray" name="lidar_sensor">
       <pose>0 0 0 0 0 0</pose>
       <visualize>true</visualize>
-      <update_rate>50</update_rate>
+      <update_rate>5</update_rate>
       <ray>
-         <scan>
-            <horizontal>
-               <samples>10</samples>
-               <resolution>1</resolution>
-               <min_angle>-0.14835</min_angle>
-               <max_angle>0.14835</max_angle>
-            </horizontal>
-            <vertical>
-               <samples>10</samples>
-               <resolution>1</resolution>
-               <min_angle>-0.14835</min_angle>
-               <max_angle>0.14835</max_angle>
-            </vertical>
-         </scan>
-         <range>
-            <min>0.01</min>
-            <max>2</max>
-            <resolution>0.02</resolution>
-         </range>
+        <scan>
+          <horizontal>
+            <samples>360</samples>
+            <resolution>1</resolution>
+            <min_angle>0.0</min_angle>
+            <max_angle>3.14159</max_angle>
+          </horizontal>
+        </scan>
+        <range>
+          <min>0.012</min>
+          <max>0.35</max>
+          <resolution>0.015</resolution>
+        </range>
+        <noise>
+          <type>gaussian</type>
+          <mean>0.0</mean>
+          <stddev>0.01</stddev>
+        </noise>
       </ray>
-      <plugin filename="libgazebo_ros_range.so" name="gazebo_ros_range">
-         <gaussianNoise>0.005</gaussianNoise>
-         <alwaysOn>true</alwaysOn>
-         <updateRate>50</updateRate>
-         <topicName>sensor/infrared</topicName>
-         <frameName>link_infrared</frameName>
-         <radiation>INFRARED</radiation>
-         <fov>0.2967</fov>
+      <plugin name="gazebo_ros_lidar_controller" filename="libgazebo_ros_laser.so">
+        <topicName>scan</topicName>
+        <frameName>link_scan</frameName>
       </plugin>
-   </sensor>
-   </gazebo>
+    </sensor>
+    <material>Gazebo/FlatBlack</material>
+  </gazebo>
+  <!-- Controller -->
+  <gazebo>
+    <plugin name="mouse_controller" filename="libgazebo_ros_diff_drive.so">
+      <commandTopic>cmd_vel</commandTopic>
+      <odometryTopic>odom</odometryTopic>
+      <odometryFrame>odom</odometryFrame>
+      <odometrySource>world</odometrySource>
+      <publishOdomTF>true</publishOdomTF>
+      <robotBaseFrame>link_chassis</robotBaseFrame>
+      <publishWheelTF>false</publishWheelTF>
+      <publishTf>true</publishTf>
+      <publishWheelJointState>true</publishWheelJointState>
+      <legacyMode>false</legacyMode>
+      <updateRate>30</updateRate>
+      <leftJoint>joint_left_wheel</leftJoint>
+      <rightJoint>joint_right_wheel</rightJoint>
+      <wheelSeparation>0.287</wheelSeparation>
+      <wheelDiameter>0.066</wheelDiameter>
+      <wheelAcceleration>1</wheelAcceleration>
+      <wheelTorque>10</wheelTorque>
+      <rosDebugLevel>na</rosDebugLevel>
+    </plugin>
+  </gazebo>
 </robot>

Commit message: Mapping

File: src/maze_generator/urdf/mouse.xacro (robot description, xacro)
@@ -89,6 +89,6 @@
     <inertial>
       <mass value="0.5"/>
-      <origin rpy="1.5707 0 1.5707" xyz="0 0 0"/>
-      <inertia ixx="0.0001062083333" ixy="0" ixz="0" iyy="0.0001416666667" iyz="0" izz="0.00003954166667"/>
+      <origin rpy="0 0 0" xyz="0 0 0"/>
+      <inertia ixx="0.00003954166667" ixy="0" ixz="0" iyy="0.0001062083333" iyz="0" izz="0.0001416666667"/>
     </inertial>
   </link>
@@ -97,5 +97,5 @@
       <mass value="0.02"/>
       <origin rpy="0 1.5707 1.5707" xyz="0 0 0"/>
-      <inertia ixx="0.000000526666666667" ixy="0" ixz="0" iyy="0.000000526666666667" iyz="0" izz="0.00000016"/>
+      <inertia ixx="5.267e-7" ixy="0" ixz="0" iyy="5.267e-7" iyz="0" izz="1e-6"/>
     </inertial>
     <collision name="link_right_wheel_collision">
@@ -124,5 +124,5 @@
       <mass value="0.02"/>
       <origin rpy="0 1.5707 1.5707" xyz="0 0 0"/>
-      <inertia ixx="0.000000526666666667" ixy="0" ixz="0" iyy="0.000000526666666667" iyz="0" izz="0.00000016"/>
+      <inertia ixx="5.267e-7" ixy="0" ixz="0" iyy="5.267e-7" iyz="0" izz="1e-6"/>
     </inertial>
     <collision name="link_left_wheel_collision">
@@ -147,31 +147,4 @@
     <joint_properties damping="1.0" friction="1.0"/>
   </joint>
-  <!-- Simulation behavior -->
-  <gazebo reference="link_left_wheel">
-    <mu1>0.1</mu1>
-    <mu2>0.1</mu2>
-    <kp>500000.0</kp>
-    <kd>10.0</kd>
-    <minDepth>0.001</minDepth>
-    <maxVel>0.1</maxVel>
-    <fdir1>1 0 0</fdir1>
-  </gazebo>
-  <gazebo reference="link_right_wheel">
-    <mu1>0.1</mu1>
-    <mu2>0.1</mu2>
-    <kp>500000.0</kp>
-    <kd>10.0</kd>
-    <minDepth>0.001</minDepth>
-    <maxVel>0.1</maxVel>
-    <fdir1>1 0 0</fdir1>
-  </gazebo>
-  <gazebo reference="link_chassis">
-    <mu1>0.1</mu1>
-    <mu2>0.1</mu2>
-    <kp>1000000.0</kp>
-    <kd>100.0</kd>
-    <minDepth>0.001</minDepth>
-    <maxVel>1.0</maxVel>
-  </gazebo>
   <!-- IMU Sensor -->
   <link name="imu_link"/>

File: src/maze_generator/urdf/mouse_ir.xacro (robot description, xacro)
@@ -89,6 +89,6 @@
     <inertial>
       <mass value="0.5"/>
-      <origin rpy="1.5707 0 1.5707" xyz="0 0 0"/>
-      <inertia ixx="0.0001062083333" ixy="0" ixz="0" iyy="0.0001416666667" iyz="0" izz="0.00003954166667"/>
+      <origin rpy="0 0 0" xyz="0 0 0"/>
+      <inertia ixx="0.00003954166667" ixy="0" ixz="0" iyy="0.0001062083333" iyz="0" izz="0.0001416666667"/>
     </inertial>
   </link>
@@ -97,5 +97,5 @@
       <mass value="0.02"/>
       <origin rpy="0 1.5707 1.5707" xyz="0 0 0"/>
-      <inertia ixx="0.000000526666666667" ixy="0" ixz="0" iyy="0.000000526666666667" iyz="0" izz="0.00000016"/>
+      <inertia ixx="5.267e-7" ixy="0" ixz="0" iyy="5.267e-7" iyz="0" izz="1e-6"/>
     </inertial>
     <collision name="link_right_wheel_collision">
@@ -124,5 +124,5 @@
       <mass value="0.02"/>
       <origin rpy="0 1.5707 1.5707" xyz="0 0 0"/>
-      <inertia ixx="0.000000526666666667" ixy="0" ixz="0" iyy="0.000000526666666667" iyz="0" izz="0.00000016"/>
+      <inertia ixx="5.267e-7" ixy="0" ixz="0" iyy="5.267e-7" iyz="0" izz="1e-6"/>
     </inertial>
     <collision name="link_left_wheel_collision">
@@ -147,31 +147,4 @@
     <joint_properties damping="1.0" friction="1.0"/>
   </joint>
-  <!-- Simulation behavior -->
-  <gazebo reference="link_left_wheel">
-    <mu1>0.1</mu1>
-    <mu2>0.1</mu2>
-    <kp>500000.0</kp>
-    <kd>10.0</kd>
-    <minDepth>0.001</minDepth>
-    <maxVel>0.1</maxVel>
-    <fdir1>1 0 0</fdir1>
-  </gazebo>
-  <gazebo reference="link_right_wheel">
-    <mu1>0.1</mu1>
-    <mu2>0.1</mu2>
-    <kp>500000.0</kp>
-    <kd>10.0</kd>
-    <minDepth>0.001</minDepth>
-    <maxVel>0.1</maxVel>
-    <fdir1>1 0 0</fdir1>
-  </gazebo>
-  <gazebo reference="link_chassis">
-    <mu1>0.1</mu1>
-    <mu2>0.1</mu2>
-    <kp>1000000.0</kp>
-    <kd>100.0</kd>
-    <minDepth>0.001</minDepth>
-    <maxVel>1.0</maxVel>
-  </gazebo>
   <!-- IMU Sensor -->
   <link name="imu_link"/>
