Commit message: change size... again....

File: src/maze_generator/urdf/mouse.xacro (robot description, xacro)
@@ -41,5 +41,5 @@
     <collision name="collision_chassis">
       <geometry>
-        <box size="0.05 0.03 0.007"/>
+        <box size="0.5 0.3 0.07"/>
       </geometry>
     </collision>
@@ -47,5 +47,5 @@
       <origin rpy="0 0 0" xyz="0 0 0"/>
       <geometry>
-        <box size="0.05 0.03 0.007"/>
+        <box size="0.5 0.3 0.07"/>
       </geometry>
       <material name="blue"/>
@@ -59,7 +59,7 @@
   <link name="link_caster">
     <collision name="caster_front_collision">
-      <origin rpy="0 0 0" xyz="0.02 0 -0.005"/>
-      <geometry>
-        <sphere radius="0.005"/>
+      <origin rpy="0 0 0" xyz="0.2 0 -0.05"/>
+      <geometry>
+        <sphere radius="0.05"/>
       </geometry>
       <surface>
@@ -75,7 +75,7 @@
     </collision>
     <visual name="caster_front_visual">
-      <origin rpy="0 0 0" xyz="0.02 0 -0.005"/>
-      <geometry>
-        <sphere radius="0.005"/>
+      <origin rpy="0 0 0" xyz="0.2 0 -0.05"/>
+      <geometry>
+        <sphere radius="0.05"/>
       </geometry>
     </visual>
@@ -88,19 +88,19 @@
   <link name="chassis_inertia">
     <inertial>
-      <mass value="0.5"/>
-      <origin rpy="1.5707 0 1.5707" xyz="0 0 0"/>
-      <inertia ixx="0.0001062083333" ixy="0" ixz="0" iyy="0.0001416666667" iyz="0" izz="0.00003954166667"/>
+      <mass value="5"/>
+      <origin rpy="0 0 0" xyz="0 0 0"/>
+      <inertia ixx="0.03954166667" ixy="0" ixz="0" iyy="0.1062083333" iyz="0" izz="0.1416666667"/>
     </inertial>
   </link>
   <link name="link_right_wheel">
     <inertial>
-      <mass value="0.02"/>
-      <origin rpy="0 1.5707 1.5707" xyz="0 0 0"/>
-      <inertia ixx="0.000000526666666667" ixy="0" ixz="0" iyy="0.000000526666666667" iyz="0" izz="0.00000016"/>
+      <mass value="0.2"/>
+      <origin rpy="0 1.5707 1.5707" xyz="0 0 0"/>
+      <inertia ixx="5.267e-4" ixy="0" ixz="0" iyy="5.267e-4" iyz="0" izz="1e-3"/>
     </inertial>
     <collision name="link_right_wheel_collision">
       <origin rpy="0 1.5707 1.5707" xyz="0 0 0"/>
       <geometry>
-        <cylinder length="0.004" radius="0.01"/>
+        <cylinder length="0.04" radius="0.1"/>
       </geometry>
     </collision>
@@ -108,10 +108,10 @@
       <origin rpy="0 1.5707 1.5707" xyz="0 0 0"/>
       <geometry>
-        <cylinder length="0.004" radius="0.01"/>
+        <cylinder length="0.04" radius="0.1"/>
       </geometry>
     </visual>
   </link>
   <joint name="joint_right_wheel" type="continuous">
-    <origin rpy="0 0 0" xyz="-0.005 0.015 0"/>
+    <origin rpy="0 0 0" xyz="-0.05 0.15 0"/>
     <child link="link_right_wheel"/>
     <parent link="link_chassis"/>
@@ -122,12 +122,12 @@
   <link name="link_left_wheel">
     <inertial>
-      <mass value="0.02"/>
-      <origin rpy="0 1.5707 1.5707" xyz="0 0 0"/>
-      <inertia ixx="0.000000526666666667" ixy="0" ixz="0" iyy="0.000000526666666667" iyz="0" izz="0.00000016"/>
+      <mass value="0.2"/>
+      <origin rpy="0 1.5707 1.5707" xyz="0 0 0"/>
+      <inertia ixx="5.267e-4" ixy="0" ixz="0" iyy="5.267e-4" iyz="0" izz="1e-3"/>
     </inertial>
     <collision name="link_left_wheel_collision">
       <origin rpy="0 1.5707 1.5707" xyz="0 0 0"/>
       <geometry>
-        <cylinder length="0.004" radius="0.01"/>
+        <cylinder length="0.04" radius="0.1"/>
       </geometry>
     </collision>
@@ -135,10 +135,10 @@
       <origin rpy="0 1.5707 1.5707" xyz="0 0 0"/>
       <geometry>
-        <cylinder length="0.004" radius="0.01"/>
+        <cylinder length="0.04" radius="0.1"/>
       </geometry>
     </visual>
   </link>
   <joint name="joint_left_wheel" type="continuous">
-    <origin rpy="0 0 0" xyz="-0.005 -0.015 0"/>
+    <origin rpy="0 0 0" xyz="-0.05 -0.15 0"/>
     <child link="link_left_wheel"/>
     <parent link="link_chassis"/>

File: src/maze_generator/urdf/mouse_ir.xacro (robot description, xacro)
@@ -41,5 +41,5 @@
     <collision name="collision_chassis">
       <geometry>
-        <box size="0.05 0.03 0.007"/>
+        <box size="0.5 0.3 0.07"/>
       </geometry>
     </collision>
@@ -47,5 +47,5 @@
       <origin rpy="0 0 0" xyz="0 0 0"/>
       <geometry>
-        <box size="0.05 0.03 0.007"/>
+        <box size="0.5 0.3 0.07"/>
       </geometry>
       <material name="blue"/>
@@ -59,7 +59,7 @@
   <link name="link_caster">
     <collision name="caster_front_collision">
-      <origin rpy="0 0 0" xyz="0.02 0 -0.005"/>
-      <geometry>
-        <sphere radius="0.005"/>
+      <origin rpy="0 0 0" xyz="0.2 0 -0.05"/>
+      <geometry>
+        <sphere radius="0.05"/>
       </geometry>
       <surface>
@@ -75,7 +75,7 @@
     </collision>
     <visual name="caster_front_visual">
-      <origin rpy="0 0 0" xyz="0.02 0 -0.005"/>
-      <geometry>
-        <sphere radius="0.005"/>
+      <origin rpy="0 0 0" xyz="0.2 0 -0.05"/>
+      <geometry>
+        <sphere radius="0.05"/>
       </geometry>
     </visual>
@@ -88,19 +88,19 @@
   <link name="chassis_inertia">
     <inertial>
-      <mass value="0.5"/>
-      <origin rpy="1.5707 0 1.5707" xyz="0 0 0"/>
-      <inertia ixx="0.0001062083333" ixy="0" ixz="0" iyy="0.0001416666667" iyz="0" izz="0.00003954166667"/>
+      <mass value="5"/>
+      <origin rpy="0 0 0" xyz="0 0 0"/>
+      <inertia ixx="0.03954166667" ixy="0" ixz="0" iyy="0.1062083333" iyz="0" izz="0.1416666667"/>
     </inertial>
   </link>
   <link name="link_right_wheel">
     <inertial>
-      <mass value="0.02"/>
-      <origin rpy="0 1.5707 1.5707" xyz="0 0 0"/>
-      <inertia ixx="0.000000526666666667" ixy="0" ixz="0" iyy="0.000000526666666667" iyz="0" izz="0.00000016"/>
+      <mass value="0.2"/>
+      <origin rpy="0 1.5707 1.5707" xyz="0 0 0"/>
+      <inertia ixx="5.267e-4" ixy="0" ixz="0" iyy="5.267e-4" iyz="0" izz="1e-3"/>
     </inertial>
     <collision name="link_right_wheel_collision">
       <origin rpy="0 1.5707 1.5707" xyz="0 0 0"/>
       <geometry>
-        <cylinder length="0.004" radius="0.01"/>
+        <cylinder length="0.04" radius="0.1"/>
       </geometry>
     </collision>
@@ -108,10 +108,10 @@
       <origin rpy="0 1.5707 1.5707" xyz="0 0 0"/>
       <geometry>
-        <cylinder length="0.004" radius="0.01"/>
+        <cylinder length="0.04" radius="0.1"/>
       </geometry>
     </visual>
   </link>
   <joint name="joint_right_wheel" type="continuous">
-    <origin rpy="0 0 0" xyz="-0.005 0.015 0"/>
+    <origin rpy="0 0 0" xyz="-0.05 0.15 0"/>
     <child link="link_right_wheel"/>
     <parent link="link_chassis"/>
@@ -122,12 +122,12 @@
   <link name="link_left_wheel">
     <inertial>
-      <mass value="0.02"/>
-      <origin rpy="0 1.5707 1.5707" xyz="0 0 0"/>
-      <inertia ixx="0.000000526666666667" ixy="0" ixz="0" iyy="0.000000526666666667" iyz="0" izz="0.00000016"/>
+      <mass value="0.2"/>
+      <origin rpy="0 1.5707 1.5707" xyz="0 0 0"/>
+      <inertia ixx="5.267e-4" ixy="0" ixz="0" iyy="5.267e-4" iyz="0" izz="1e-3"/>
     </inertial>
     <collision name="link_left_wheel_collision">
       <origin rpy="0 1.5707 1.5707" xyz="0 0 0"/>
       <geometry>
-        <cylinder length="0.004" radius="0.01"/>
+        <cylinder length="0.04" radius="0.1"/>
       </geometry>
     </collision>
@@ -135,10 +135,10 @@
       <origin rpy="0 1.5707 1.5707" xyz="0 0 0"/>
       <geometry>
-        <cylinder length="0.004" radius="0.01"/>
+        <cylinder length="0.04" radius="0.1"/>
       </geometry>
     </visual>
   </link>
   <joint name="joint_left_wheel" type="continuous">
-    <origin rpy="0 0 0" xyz="-0.005 -0.015 0"/>
+    <origin rpy="0 0 0" xyz="-0.05 -0.15 0"/>
     <child link="link_left_wheel"/>
     <parent link="link_chassis"/>
@@ -218,5 +218,5 @@
   <!-- IR Sensor -->
   <joint name="fixed_sensor" type="fixed">
-    <origin rpy="0 0 0" xyz="0.0275 0 0"/>
+    <origin rpy="0 0 0" xyz="0.275 0 0"/>
     <child link="link_infrared"/>
     <parent link="link_chassis"/>
@@ -226,5 +226,5 @@
       <origin rpy="0 0 0" xyz="0 0 0"/>
       <geometry>
-        <box size="0.005 0.005 0.005"/>
+        <box size="0.05 0.05 0.05"/>
       </geometry>
     </visual>

File: src/maze_generator/urdf/mouse_lidar.xacro (robot description, xacro)
@@ -41,5 +41,5 @@
     <collision name="collision_chassis">
       <geometry>
-        <box size="0.05 0.03 0.007"/>
+        <box size="0.5 0.3 0.07"/>
       </geometry>
     </collision>
@@ -47,5 +47,5 @@
       <origin rpy="0 0 0" xyz="0 0 0"/>
       <geometry>
-        <box size="0.05 0.03 0.007"/>
+        <box size="0.5 0.3 0.07"/>
       </geometry>
       <material name="blue"/>
@@ -59,7 +59,7 @@
   <link name="chassis_inertia">
     <inertial>
-      <mass value="0.5"/>
+      <mass value="5"/>
       <origin rpy="0 0 0" xyz="0 0 0"/>
-      <inertia ixx="0.00003954166667" ixy="0" ixz="0" iyy="0.0001062083333" iyz="0" izz="0.0001416666667"/>
+      <inertia ixx="0.03954166667" ixy="0" ixz="0" iyy="0.1062083333" iyz="0" izz="0.1416666667"/>
     </inertial>
   </link>
@@ -71,7 +71,7 @@
   <link name="link_caster">
     <collision name="caster_front_collision">
-      <origin rpy="0 0 0" xyz="0.02 0 -0.005"/>
-      <geometry>
-        <sphere radius="0.005"/>
+      <origin rpy="0 0 0" xyz="0.2 0 -0.05"/>
+      <geometry>
+        <sphere radius="0.05"/>
       </geometry>
       <surface>
@@ -87,7 +87,7 @@
     </collision>
     <visual name="caster_front_visual">
-      <origin rpy="0 0 0" xyz="0.02 0 -0.005"/>
-      <geometry>
-        <sphere radius="0.005"/>
+      <origin rpy="0 0 0" xyz="0.2 0 -0.05"/>
+      <geometry>
+        <sphere radius="0.05"/>
       </geometry>
     </visual>
@@ -95,12 +95,12 @@
   <link name="link_right_wheel">
     <inertial>
-      <mass value="0.02"/>
-      <origin rpy="0 1.5707 1.5707" xyz="0 0 0"/>
-      <inertia ixx="5.267e-7" ixy="0" ixz="0" iyy="5.267e-7" iyz="0" izz="1e-6"/>
+      <mass value="0.2"/>
+      <origin rpy="0 1.5707 1.5707" xyz="0 0 0"/>
+      <inertia ixx="5.267e-4" ixy="0" ixz="0" iyy="5.267e-4" iyz="0" izz="1e-3"/>
     </inertial>
     <collision name="link_right_wheel_collision">
       <origin rpy="0 1.5707 1.5707" xyz="0 0 0"/>
       <geometry>
-        <cylinder length="0.004" radius="0.01"/>
+        <cylinder length="0.04" radius="0.1"/>
       </geometry>
     </collision>
@@ -108,10 +108,10 @@
       <origin rpy="0 1.5707 1.5707" xyz="0 0 0"/>
       <geometry>
-        <cylinder length="0.004" radius="0.01"/>
+        <cylinder length="0.04" radius="0.1"/>
       </geometry>
     </visual>
   </link>
   <joint name="joint_right_wheel" type="continuous">
-    <origin rpy="0 0 0" xyz="-0.005 0.015 0"/>
+    <origin rpy="0 0 0" xyz="-0.05 0.15 0"/>
     <child link="link_right_wheel"/>
     <parent link="link_chassis"/>
@@ -122,12 +122,12 @@
   <link name="link_left_wheel">
     <inertial>
-      <mass value="0.02"/>
-      <origin rpy="0 1.5707 1.5707" xyz="0 0 0"/>
-      <inertia ixx="5.267e-7" ixy="0" ixz="0" iyy="5.267e-7" iyz="0" izz="1e-6"/>
+      <mass value="0.2"/>
+      <origin rpy="0 1.5707 1.5707" xyz="0 0 0"/>
+      <inertia ixx="5.267e-4" ixy="0" ixz="0" iyy="5.267e-4" iyz="0" izz="1e-3"/>
     </inertial>
     <collision name="link_left_wheel_collision">
       <origin rpy="0 1.5707 1.5707" xyz="0 0 0"/>
       <geometry>
-        <cylinder length="0.004" radius="0.01"/>
+        <cylinder length="0.04" radius="0.1"/>
       </geometry>
     </collision>
@@ -135,10 +135,10 @@
       <origin rpy="0 1.5707 1.5707" xyz="0 0 0"/>
       <geometry>
-        <cylinder length="0.004" radius="0.01"/>
+        <cylinder length="0.04" radius="0.1"/>
       </geometry>
     </visual>
   </link>
   <joint name="joint_left_wheel" type="continuous">
-    <origin rpy="0 0 0" xyz="-0.005 -0.015 0"/>
+    <origin rpy="0 0 0" xyz="-0.05 -0.15 0"/>
     <child link="link_left_wheel"/>
     <parent link="link_chassis"/>
@@ -193,5 +193,5 @@
     <parent link="link_chassis"/>
     <child link="link_scan"/>
-    <origin xyz="0.015 0 0.006" rpy="0 0 -1.57079"/>
+    <origin xyz="0.15 0 0.06" rpy="0 0 -1.57079"/>
   </joint>
   <link name="link_scan">
@@ -199,5 +199,5 @@
       <origin xyz="0 0 0" rpy="0 0 0"/>
       <geometry>
-        <box size="0.005 0.005 0.005"/>
+        <box size="0.05 0.05 0.05"/>
       </geometry>
       <material name="black"/>
@@ -206,5 +206,5 @@
       <origin xyz="0 0 0" rpy="0 0 0"/>
       <geometry>
-        <box size="0.005 0.005 0.005"/>
+        <box size="0.05 0.05 0.05"/>
       </geometry>
     </collision>

Commit message: colors

File: src/maze_generator/urdf/mouse.xacro (robot description, xacro)
@@ -25,15 +25,21 @@
     <color rgba="1.0 1.0 1.0 1.0"/>
   </material>
+  <material name="pantone202RAS">
+    <color rgba="0.59608 0.0 0.18039 1.0"/>
+  </material>
+  <material name="pantone2623RAS">
+    <color rgba="0.38039 0.66667 0.415686 1.0"/>
+  </material>
   <gazebo reference="link_chassis">
-    <material>Gazebo/Orange</material>
+    <material>Gazebo/pantone202RAS</material>
   </gazebo>
   <gazebo reference="link_caster">
-    <material>Gazebo/Gray</material>
+    <material>Gazebo/pantone2623RAS</material>
   </gazebo>
   <gazebo reference="link_left_wheel">
-    <material>Gazebo/Blue</material>
+    <material>Gazebo/pantone2623RAS</material>
   </gazebo>
   <gazebo reference="link_right_wheel">
-    <material>Gazebo/Blue</material>
+    <material>Gazebo/pantone2623RAS</material>
   </gazebo>
   <!-- Robot description -->
@@ -49,5 +55,5 @@
         <box size="0.5 0.3 0.07"/>
       </geometry>
-      <material name="blue"/>
+      <material name="pantone202RAS"/>
     </visual>
   </link>

Commit message: Back

File: src/maze_generator/urdf/mouse.xacro (robot description, xacro)
@@ -25,21 +25,15 @@
     <color rgba="1.0 1.0 1.0 1.0"/>
   </material>
-  <material name="pantone202RAS">
-    <color rgba="0.59608 0.0 0.18039 1.0"/>
-  </material>
-  <material name="pantone2623RAS">
-    <color rgba="0.38039 0.66667 0.415686 1.0"/>
-  </material>
   <gazebo reference="link_chassis">
-    <material>Gazebo/pantone202RAS</material>
+    <material>Gazebo/Orange</material>
   </gazebo>
   <gazebo reference="link_caster">
-    <material>Gazebo/pantone2623RAS</material>
+    <material>Gazebo/Gray</material>
   </gazebo>
   <gazebo reference="link_left_wheel">
-    <material>Gazebo/pantone2623RAS</material>
+    <material>Gazebo/Blue</material>
   </gazebo>
   <gazebo reference="link_right_wheel">
-    <material>Gazebo/pantone2623RAS</material>
+    <material>Gazebo/Blue</material>
   </gazebo>
   <!-- Robot description -->
@@ -55,5 +49,5 @@
         <box size="0.5 0.3 0.07"/>
       </geometry>
-      <material name="pantone202RAS"/>
+      <material name="blue"/>
     </visual>
   </link>
