Commit message: Better meshes

File: src/maze_generator/urdf/mouse.xacro (robot description, xacro)
@@ -37,9 +37,14 @@
     <material>Gazebo/Blue</material>
   </gazebo>
-  <!-- Robot description -->
-  <link name="link_chassis">
+  <!-- =========================================== -->
+  <!-- ROBOT DESCRIPTION -->
+  <!-- =========================================== -->
+  <!-- Chassis -->
+  <link name="chassis_base">
     <collision name="collision_chassis">
-      <geometry>
-        <box size="0.5 0.3 0.07"/>
+      <origin rpy="0 0 0" xyz="0 0 0"/>
+      <geometry>
+        <box size="0.48 0.48 0.012"/>
+        <!--mesh filename="package://maze_generator/urdf/meshes/umouse_v2_base.stl" scale="0.003 0.003 0.003"/-->
       </geometry>
     </collision>
@@ -47,100 +52,167 @@
       <origin rpy="0 0 0" xyz="0 0 0"/>
       <geometry>
-        <box size="0.5 0.3 0.07"/>
+        <box size="0.48 0.48 0.012"/>
+        <!--mesh filename="package://maze_generator/urdf/meshes/umouse_v2_base.stl" scale="0.003 0.003 0.003"/-->
       </geometry>
       <material name="blue"/>
     </visual>
   </link>
-  <joint name="fixed_caster_joint" type="fixed">
+  <joint name="fixed_inertia" type="fixed">
     <origin rpy="0 0 0" xyz="0 0 0"/>
-    <child link="link_caster"/>
-    <parent link="link_chassis"/>
-  </joint>
-  <link name="link_caster">
-    <collision name="caster_front_collision">
-      <origin rpy="0 0 0" xyz="0.2 0 -0.05"/>
-      <geometry>
-        <sphere radius="0.05"/>
-      </geometry>
-      <surface>
-        <friction>
-          <ode>
-            <mu>0</mu>
-            <mu2>0</mu2>
-            <slip1>1.0</slip1>
-            <slip2>1.0</slip2>
-          </ode>
-        </friction>
-      </surface>
-    </collision>
-    <visual name="caster_front_visual">
-      <origin rpy="0 0 0" xyz="0.2 0 -0.05"/>
-      <geometry>
-        <sphere radius="0.05"/>
-      </geometry>
-    </visual>
-  </link>
-  <joint name="fixed_base_joint" type="fixed">
+    <parent link="chassis_base"/>
+    <child link="chassis_inertia"/>
+  </joint>
+  <link name="chassis_inertia">
+    <inertial>
+      <mass value="0.2"/>
+      <origin rpy="0 0 0" xyz="0 0 0.36"/>
+      <inertia ixx="0.0038424" ixy="0" ixz="0" iyy="0.0038424" iyz="0" izz="0.00768"/>
+    </inertial>
+  </link>
+  <link name="chassis_sensors">
+    <inertial>
+      <mass value="0.5"/>
+      <origin rpy="0 0 0" xyz="0 0 0"/>
+      <inertia ixx="0.003" ixy="0" ixz="0" iyy="0.0048" iyz="0" izz="0.003"/>
+    </inertial>
+    <collision name="collision_chassis">
+      <origin rpy="0 0 0" xyz="0 0 0.105"/>
+      <geometry>
+        <box size="0.48 0.48 0.21"/>
+        <!--mesh filename="package://maze_generator/urdf/meshes/umouse_v2_lidar.stl" scale="0.003 0.003 0.003"/-->
+      </geometry>
+    </collision>
+    <collision name="collision_chassis">
+      <origin rpy="0 0 0" xyz="0.06 0 0.28"/>
+      <geometry>
+        <box size="0.2955 0.21 0.16"/>
+        <!--mesh filename="package://maze_generator/urdf/meshes/umouse_v2_lidar.stl" scale="0.003 0.003 0.003"/-->
+      </geometry>
+    </collision>
+    <visual>
+      <origin rpy="0 0 0" xyz="0 0 0"/>
+      <geometry>
+        <!--box size="0.48 0.48 0.21"/-->
+        <mesh filename="package://maze_generator/urdf/meshes/umouse_v2_lidar.stl" scale="0.003 0.003 0.003"/>
+      </geometry>
+      <material name="blue"/>
+    </visual>
+  </link>
+  <joint name="fixed_base" type="fixed">
     <origin rpy="0 0 0" xyz="0 0 0"/>
-    <child link="chassis_inertia"/>
-    <parent link="link_chassis"/>
-  </joint>
-  <link name="chassis_inertia">
-    <inertial>
-      <mass value="5"/>
-      <origin rpy="0 0 0" xyz="0 0 0"/>
-      <inertia ixx="0.03954166667" ixy="0" ixz="0" iyy="0.1062083333" iyz="0" izz="0.1416666667"/>
-    </inertial>
-  </link>
+    <parent link="chassis_base"/>
+    <child link="chassis_sensors"/>
+  </joint>
+  <!-- Front castor wheel -->
+  <link name="fcastor_wheel">
+    <visual>
+      <origin rpy="0 0 0" xyz="0 0 0"/>
+      <geometry>
+        <sphere radius="0.0191"/>
+        <!--mesh filename="package://maze_generator/urdf/meshes/umouse_v2_casterball.stl" scale="0.003 0.003 0.003"/-->
+      </geometry>
+    </visual>
+    <collision>
+      <origin rpy="0 0 0" xyz="0 0 -0.024"/>
+      <geometry>
+        <sphere radius="0.0191"/>
+        <!--mesh filename="package://maze_generator/urdf/meshes/umouse_v2_casterball.stl" scale="0.003 0.003 0.003"/-->
+      </geometry>
+    </collision>
+    <inertial>
+      <origin rpy="0 0 0" xyz="0 0 0"/>
+      <mass value="0.1" />
+      <inertia ixx="0.000014516" ixy="0.0" ixz="0.0" iyy="0.000014516" iyz="0.0" izz="0.000014516"/>
+    </inertial>
+  </link>
+  <joint name="base__fcastor_wheel" type="continuous">
+    <parent link="chassis_base"/>
+    <child link="fcastor_wheel"/>
+    <origin xyz="0.21 0 -0.012" rpy="0 0 0"/>
+    <axis xyz="0 0 1"/>
+  </joint>
+  <!-- Back castor wheel -->
+  <link name="bcastor_wheel">
+    <visual>
+      <origin rpy="0 0 0" xyz="0 0 0"/>
+      <geometry>
+        <sphere radius="0.0191"/>
+        <!--mesh filename="package://maze_generator/urdf/meshes/umouse_v2_casterball.stl" scale="0.003 0.003 0.003"/-->
+      </geometry>
+    </visual>
+    <collision>
+      <origin rpy="0 0 0" xyz="0 0 -0.024"/>
+      <geometry>
+        <sphere radius="0.0191"/>
+        <!--mesh filename="package://maze_generator/urdf/meshes/umouse_v2_casterball.stl" scale="0.003 0.003 0.003"/-->
+      </geometry>
+    </collision>
+    <inertial>
+      <mass value="0.1" />
+      <inertia ixx="0.000014516" ixy="0.0" ixz="0.0" iyy="0.000014516" iyz="0.0" izz="0.000014516"/>
+    </inertial>
+  </link>
+  <joint name="base__bcastor_wheel" type="continuous">
+    <parent link="chassis_base"/>
+    <child link="bcastor_wheel"/>
+    <origin xyz="-0.21 0 -0.012" rpy="0 0 0"/>
+    <axis xyz="0 0 1"/>
+  </joint>
+  <!-- Right wheel -->
   <link name="link_right_wheel">
     <inertial>
-      <mass value="0.2"/>
-      <origin rpy="0 1.5707 1.5707" xyz="0 0 0"/>
-      <inertia ixx="5.267e-4" ixy="0" ixz="0" iyy="5.267e-4" iyz="0" izz="1e-3"/>
+      <mass value="0.12"/>
+      <origin rpy="0 1.5707 -1.5707" xyz="0 0.015 0"/>
+      <inertia ixx="0.000252" ixy="0" ixz="0" iyy="0.000252" iyz="0" izz="0.000486"/>
     </inertial>
     <collision name="link_right_wheel_collision">
-      <origin rpy="0 1.5707 1.5707" xyz="0 0 0"/>
-      <geometry>
-        <cylinder length="0.04" radius="0.1"/>
+      <origin rpy="0 1.570796 1.570796" xyz="0 0.015 0"/>
+      <geometry>
+        <cylinder length="0.03" radius="0.09"/>
+        <!--mesh filename="package://maze_generator/urdf/meshes/umouse_v2_wheel.stl" scale="0.003 0.003 0.003"/-->
       </geometry>
     </collision>
     <visual name="link_right_wheel_visual">
-      <origin rpy="0 1.5707 1.5707" xyz="0 0 0"/>
-      <geometry>
-        <cylinder length="0.04" radius="0.1"/>
+      <origin rpy="0 0 3.141592" xyz="0 0 0"/>
+      <geometry>
+        <!--cylinder length="0.03" radius="0.09"/-->
+        <mesh filename="package://maze_generator/urdf/meshes/umouse_v2_wheel.stl" scale="0.003 0.003 0.003"/>
       </geometry>
     </visual>
   </link>
   <joint name="joint_right_wheel" type="continuous">
-    <origin rpy="0 0 0" xyz="-0.05 0.15 0"/>
+    <origin rpy="0 0 0" xyz="0 0.219 0.0345"/>
     <child link="link_right_wheel"/>
-    <parent link="link_chassis"/>
+    <parent link="chassis_base"/>
     <axis rpy="0 0 0" xyz="0 1 0"/>
     <limit effort="10000" velocity="1000"/>
     <joint_properties damping="1.0" friction="1.0"/>
   </joint>
+  <!-- Left wheel -->
   <link name="link_left_wheel">
     <inertial>
-      <mass value="0.2"/>
-      <origin rpy="0 1.5707 1.5707" xyz="0 0 0"/>
-      <inertia ixx="5.267e-4" ixy="0" ixz="0" iyy="5.267e-4" iyz="0" izz="1e-3"/>
+      <mass value="0.12"/>
+      <origin rpy="0 1.5707 -1.5707" xyz="0 -0.015 0"/>
+      <inertia ixx="0.000252" ixy="0" ixz="0" iyy="0.000252" iyz="0" izz="0.000486"/>
     </inertial>
     <collision name="link_left_wheel_collision">
-      <origin rpy="0 1.5707 1.5707" xyz="0 0 0"/>
-      <geometry>
-        <cylinder length="0.04" radius="0.1"/>
+      <origin rpy="0 1.570796 1.570796" xyz="0 -0.015 0"/>
+      <geometry>
+        <cylinder length="0.03" radius="0.09"/>
+        <!--mesh filename="package://maze_generator/urdf/meshes/umouse_v2_wheel.stl" scale="0.003 0.003 0.003"/-->
       </geometry>
     </collision>
     <visual name="link_left_wheel_visual">
-      <origin rpy="0 1.5707 1.5707" xyz="0 0 0"/>
-      <geometry>
-        <cylinder length="0.04" radius="0.1"/>
+      <origin rpy="0 0 0" xyz="0 0 0"/>
+      <geometry>
+        <!--cylinder length="0.03" radius="0.09"/-->
+        <mesh filename="package://maze_generator/urdf/meshes/umouse_v2_wheel.stl" scale="0.003 0.003 0.003"/>
       </geometry>
     </visual>
   </link>
   <joint name="joint_left_wheel" type="continuous">
-    <origin rpy="0 0 0" xyz="-0.05 -0.15 0"/>
+    <origin rpy="0 0 0" xyz="0 -0.219 0.0345"/>
     <child link="link_left_wheel"/>
-    <parent link="link_chassis"/>
+    <parent link="chassis_base"/>
     <axis rpy="0 0 0" xyz="0 1 0"/>
     <limit effort="10000" velocity="1000"/>
@@ -150,5 +222,5 @@
   <link name="imu_link"/>
   <joint name="imu_joint" type="fixed">
-    <parent link="link_chassis"/>
+    <parent link="chassis_base"/>
     <child link="imu_link"/>
     <origin xyz="0 0 0" rpy="0 0 0"/>
@@ -189,4 +261,57 @@
     </plugin>
   </gazebo>
+  <!-- LiDAR Sensor -->
+  <joint name="scan_joint" type="fixed">
+    <parent link="chassis_base"/>
+    <child link="link_scan"/>
+    <origin xyz="0.15 0 0.31" rpy="0 0 -1.57079"/>
+  </joint>
+  <link name="link_scan">
+  <!--  <visual>
+      <origin xyz="0 0 0" rpy="0 0 0"/>
+      <geometry>
+        <box size="0.05 0.05 0.05"/>
+      </geometry>
+      <material name="black"/>
+    </visual>
+    <collision>
+      <origin xyz="0 0 0" rpy="0 0 0"/>
+      <geometry>
+        <box size="0.05 0.05 0.05"/>
+      </geometry>
+    </collision> -->
+  </link>
+  <gazebo reference="link_scan">
+    <sensor type="ray" name="lidar_sensor">
+      <pose>0 0 0 0 0 0</pose>
+      <visualize>true</visualize>
+      <update_rate>5</update_rate>
+      <ray>
+        <scan>
+          <horizontal>
+            <samples>360</samples>
+            <resolution>1</resolution>
+            <min_angle>0.0</min_angle>
+            <max_angle>3.14159</max_angle>
+          </horizontal>
+        </scan>
+        <range>
+          <min>0.12</min>
+          <max>4.8</max>
+          <resolution>0.015</resolution>
+        </range>
+        <noise>
+          <type>gaussian</type>
+          <mean>0.0</mean>
+          <stddev>0.01</stddev>
+        </noise>
+      </ray>
+      <plugin name="gazebo_ros_lidar_controller" filename="libgazebo_ros_laser.so">
+        <topicName>scan</topicName>
+        <frameName>link_scan</frameName>
+      </plugin>
+    </sensor>
+    <material>Gazebo/FlatBlack</material>
+  </gazebo>
   <!-- Controller -->
   <gazebo>
@@ -205,8 +330,8 @@
       <leftJoint>joint_left_wheel</leftJoint>
       <rightJoint>joint_right_wheel</rightJoint>
-      <wheelSeparation>0.287</wheelSeparation>
-      <wheelDiameter>0.066</wheelDiameter>
-      <wheelAcceleration>1</wheelAcceleration>
-      <wheelTorque>10</wheelTorque>
+      <wheelSeparation>0.4380</wheelSeparation>
+      <wheelDiameter>0.18</wheelDiameter>
+      <wheelAcceleration>3</wheelAcceleration>
+      <wheelTorque>50</wheelTorque>
       <rosDebugLevel>na</rosDebugLevel>
     </plugin>

Commit message: Meshes

File: src/maze_generator/urdf/mouse.xacro (robot description, xacro)
@@ -80,5 +80,5 @@
       <geometry>
         <box size="0.48 0.48 0.21"/>
-        <!--mesh filename="package://maze_generator/urdf/meshes/umouse_v2_lidar.stl" scale="0.003 0.003 0.003"/-->
+        <!--mesh filename="package://maze_generator/urdf/meshes/umouse_lidar.stl" scale="0.003 0.003 0.003"/-->
       </geometry>
     </collision>
@@ -87,5 +87,5 @@
       <geometry>
         <box size="0.2955 0.21 0.16"/>
-        <!--mesh filename="package://maze_generator/urdf/meshes/umouse_v2_lidar.stl" scale="0.003 0.003 0.003"/-->
+        <!--mesh filename="package://maze_generator/urdf/meshes/umouse_lidar.stl" scale="0.003 0.003 0.003"/-->
       </geometry>
     </collision>
@@ -94,5 +94,5 @@
       <geometry>
         <!--box size="0.48 0.48 0.21"/-->
-        <mesh filename="package://maze_generator/urdf/meshes/umouse_v2_lidar.stl" scale="0.003 0.003 0.003"/>
+        <mesh filename="package://maze_generator/urdf/meshes/umouse_lidar.stl" scale="0.003 0.003 0.003"/>
       </geometry>
       <material name="blue"/>
@@ -170,5 +170,5 @@
       <geometry>
         <cylinder length="0.03" radius="0.09"/>
-        <!--mesh filename="package://maze_generator/urdf/meshes/umouse_v2_wheel.stl" scale="0.003 0.003 0.003"/-->
+        <!--mesh filename="package://maze_generator/urdf/meshes/umouse_wheel.stl" scale="0.003 0.003 0.003"/-->
       </geometry>
     </collision>
@@ -177,5 +177,5 @@
       <geometry>
         <!--cylinder length="0.03" radius="0.09"/-->
-        <mesh filename="package://maze_generator/urdf/meshes/umouse_v2_wheel.stl" scale="0.003 0.003 0.003"/>
+        <mesh filename="package://maze_generator/urdf/meshes/umouse_wheel.stl" scale="0.003 0.003 0.003"/>
       </geometry>
     </visual>
@@ -200,5 +200,5 @@
       <geometry>
         <cylinder length="0.03" radius="0.09"/>
-        <!--mesh filename="package://maze_generator/urdf/meshes/umouse_v2_wheel.stl" scale="0.003 0.003 0.003"/-->
+        <!--mesh filename="package://maze_generator/urdf/meshes/umouse_wheel.stl" scale="0.003 0.003 0.003"/-->
       </geometry>
     </collision>
@@ -207,5 +207,5 @@
       <geometry>
         <!--cylinder length="0.03" radius="0.09"/-->
-        <mesh filename="package://maze_generator/urdf/meshes/umouse_v2_wheel.stl" scale="0.003 0.003 0.003"/>
+        <mesh filename="package://maze_generator/urdf/meshes/umouse_wheel.stl" scale="0.003 0.003 0.003"/>
       </geometry>
     </visual>
@@ -332,6 +332,6 @@
       <wheelSeparation>0.4380</wheelSeparation>
       <wheelDiameter>0.18</wheelDiameter>
-      <wheelAcceleration>3</wheelAcceleration>
-      <wheelTorque>50</wheelTorque>
+      <wheelAcceleration>1</wheelAcceleration>
+      <wheelTorque>30</wheelTorque>
       <rosDebugLevel>na</rosDebugLevel>
     </plugin>
