Commit message: Mesh fix

File: src/maze_generator/urdf/mouse_lidar.xacro (robot description, xacro)
@@ -37,9 +37,13 @@
     <material>Gazebo/Blue</material>
   </gazebo>
-  <!-- Robot description -->
-  <link name="link_chassis">
+  <!-- =========================================== -->
+  <!-- ROBOT DESCRIPTION -->
+  <!-- =========================================== -->
+  <!-- Chassis -->
+  <link name="chassis_base">
     <collision name="collision_chassis">
-      <geometry>
-        <box size="0.5 0.3 0.07"/>
+      <origin rpy="0 0 0" xyz="0 0 -0.006"/>
+      <geometry>
+        <box size="0.48 0.48 0.012"/>
       </geometry>
     </collision>
@@ -47,100 +51,168 @@
       <origin rpy="0 0 0" xyz="0 0 0"/>
       <geometry>
-        <box size="0.5 0.3 0.07"/>
+        <mesh filename="package://maze_generator/urdf/meshes/umouse_base.stl" scale="0.003 0.003 0.003"/>
       </geometry>
       <material name="blue"/>
     </visual>
   </link>
-  <joint name="fixed_base_joint" type="fixed">
+  <link name="chassis_inertia">
+    <inertial>
+      <mass value="0.2"/>
+      <origin rpy="0 0 0" xyz="0 0 -0.006"/>
+      <inertia ixx="0.0038424" ixy="0" ixz="0" iyy="0.0038424" iyz="0" izz="0.00768"/>
+    </inertial>
+  </link>
+  <joint name="fixed_inertia" type="fixed">
     <origin rpy="0 0 0" xyz="0 0 0"/>
+    <parent link="chassis_base"/>
     <child link="chassis_inertia"/>
-    <parent link="link_chassis"/>
-  </joint>
-  <link name="chassis_inertia">
-    <inertial>
-      <mass value="5"/>
+  </joint>
+  <link name="chassis_sensors">
+    <inertial>
+      <mass value="0.5"/>
+      <origin rpy="0 0 0" xyz="0 0 0.096"/>
+      <inertia ixx="0.011136" ixy="0" ixz="0" iyy="0.011136" iyz="0" izz="0.0192"/>
+    </inertial>
+    <collision name="collision_chassis">
+      <origin rpy="0 0 0" xyz="0 0 0.096"/>
+      <geometry>
+        <box size="0.48 0.48 0.192"/>
+      </geometry>
+    </collision>
+    <visual>
       <origin rpy="0 0 0" xyz="0 0 0"/>
-      <inertia ixx="0.03954166667" ixy="0" ixz="0" iyy="0.1062083333" iyz="0" izz="0.1416666667"/>
-    </inertial>
-  </link>
-  <joint name="fixed_caster_joint" type="fixed">
+      <geometry>
+        <mesh filename="package://maze_generator/urdf/meshes/umouse_lidar.stl" scale="0.003 0.003 0.003"/>
+      </geometry>
+      <material name="blue"/>
+    </visual>
+  </link>
+  <joint name="fixed_base" type="fixed">
     <origin rpy="0 0 0" xyz="0 0 0"/>
-    <child link="link_caster"/>
-    <parent link="link_chassis"/>
-  </joint>
-  <link name="link_caster">
-    <collision name="caster_front_collision">
-      <origin rpy="0 0 0" xyz="0.2 0 -0.05"/>
-      <geometry>
-        <sphere radius="0.05"/>
-      </geometry>
-      <surface>
-        <friction>
-          <ode>
-            <mu>0</mu>
-            <mu2>0</mu2>
-            <slip1>1.0</slip1>
-            <slip2>1.0</slip2>
-          </ode>
-        </friction>
-      </surface>
-    </collision>
-    <visual name="caster_front_visual">
-      <origin rpy="0 0 0" xyz="0.2 0 -0.05"/>
-      <geometry>
-        <sphere radius="0.05"/>
-      </geometry>
-    </visual>
-  </link>
+    <parent link="chassis_base"/>
+    <child link="chassis_sensors"/>
+  </joint>
+  <link name="sensor_lidar">
+    <inertial>
+      <mass value="0.19"/>
+      <origin rpy="0 0 0" xyz="0 0 0"/>
+      <inertia ixx="0.00121125" ixy="0" ixz="0" iyy="0.001799063" iyz="0" izz="0.001984313"/>
+    </inertial>
+    <collision>
+      <origin xyz="0 0 0" rpy="0 0 0"/>
+      <geometry>
+        <box size="0.285 0.21 0.18"/>
+      </geometry>
+    </collision>
+  </link>
+  <joint name="fixed_sensor" type="fixed">
+    <origin rpy="0 0 0" xyz="0.06225 0 0.28"/>
+    <parent link="chassis_sensors"/>
+    <child link="sensor_lidar"/>
+  </joint>
+  <!-- Front castor wheel -->
+  <link name="fcastor_wheel">
+    <visual>
+      <origin rpy="0 0 0" xyz="0 0 -0.012"/>
+      <geometry>
+        <mesh filename="package://maze_generator/urdf/meshes/umouse_casterball.stl" scale="0.003 0.003 0.003"/>
+      </geometry>
+    </visual>
+    <collision>
+      <origin rpy="0 0 0" xyz="0 0 -0.03375"/>
+      <geometry>
+        <sphere radius="0.02175"/>
+      </geometry>
+    </collision>
+    <inertial>
+      <origin rpy="0 0 0" xyz="0 0 -0.03375"/>
+      <mass value="0.1" />
+      <inertia ixx="0.000014516" ixy="0.0" ixz="0.0" iyy="0.000014516" iyz="0.0" izz="0.000014516"/>
+    </inertial>
+  </link>
+  <joint name="base__fcastor_wheel" type="continuous">
+    <parent link="chassis_base"/>
+    <child link="fcastor_wheel"/>
+    <origin xyz="0.21 0 0" rpy="0 0 0"/>
+    <axis xyz="0 0 1"/>
+  </joint>
+  <!-- Back castor wheel -->
+  <link name="bcastor_wheel">
+    <visual>
+      <origin rpy="0 0 0" xyz="0 0 -0.012"/>
+      <geometry>
+        <mesh filename="package://maze_generator/urdf/meshes/umouse_casterball.stl" scale="0.003 0.003 0.003"/>
+      </geometry>
+    </visual>
+    <collision>
+      <origin rpy="0 0 0" xyz="0 0 -0.03375"/>
+      <geometry>
+        <sphere radius="0.02175"/>
+      </geometry>
+    </collision>
+    <inertial>
+      <origin rpy="0 0 0" xyz="0 0 -0.03375"/>
+      <mass value="0.1" />
+      <inertia ixx="0.000014516" ixy="0.0" ixz="0.0" iyy="0.000014516" iyz="0.0" izz="0.000014516"/>
+    </inertial>
+  </link>
+  <joint name="base__bcastor_wheel" type="continuous">
+    <parent link="chassis_base"/>
+    <child link="bcastor_wheel"/>
+    <origin xyz="-0.21 0 0" rpy="0 0 0"/>
+    <axis xyz="0 0 1"/>
+  </joint>
+  <!-- Right wheel -->
   <link name="link_right_wheel">
     <inertial>
-      <mass value="0.2"/>
-      <origin rpy="0 1.5707 1.5707" xyz="0 0 0"/>
-      <inertia ixx="5.267e-4" ixy="0" ixz="0" iyy="5.267e-4" iyz="0" izz="1e-3"/>
+      <mass value="0.12"/>
+      <origin rpy="0 1.5707 -1.5707" xyz="0 0 0"/>
+      <inertia ixx="0.000252" ixy="0" ixz="0" iyy="0.000252" iyz="0" izz="0.000486"/>
     </inertial>
     <collision name="link_right_wheel_collision">
-      <origin rpy="0 1.5707 1.5707" xyz="0 0 0"/>
-      <geometry>
-        <cylinder length="0.04" radius="0.1"/>
+      <origin rpy="0 1.570796 1.570796" xyz="0 0 0"/>
+      <geometry>
+        <cylinder length="0.03" radius="0.09"/>
       </geometry>
     </collision>
     <visual name="link_right_wheel_visual">
-      <origin rpy="0 1.5707 1.5707" xyz="0 0 0"/>
-      <geometry>
-        <cylinder length="0.04" radius="0.1"/>
+      <origin rpy="0 0 -1.570796" xyz="0 0 0"/>
+      <geometry>
+        <mesh filename="package://maze_generator/urdf/meshes/umouse_wheel.stl" scale="0.003 0.003 0.003"/>
       </geometry>
     </visual>
   </link>
   <joint name="joint_right_wheel" type="continuous">
-    <origin rpy="0 0 0" xyz="-0.05 0.15 0"/>
+    <origin rpy="0 0 0" xyz="0 0.231 0.0345"/>
     <child link="link_right_wheel"/>
-    <parent link="link_chassis"/>
+    <parent link="chassis_base"/>
     <axis rpy="0 0 0" xyz="0 1 0"/>
     <limit effort="10000" velocity="1000"/>
     <joint_properties damping="1.0" friction="1.0"/>
   </joint>
+  <!-- Left wheel -->
   <link name="link_left_wheel">
     <inertial>
-      <mass value="0.2"/>
-      <origin rpy="0 1.5707 1.5707" xyz="0 0 0"/>
-      <inertia ixx="5.267e-4" ixy="0" ixz="0" iyy="5.267e-4" iyz="0" izz="1e-3"/>
+      <mass value="0.12"/>
+      <origin rpy="0 1.5707 -1.5707" xyz="0 0 0"/>
+      <inertia ixx="0.000252" ixy="0" ixz="0" iyy="0.000252" iyz="0" izz="0.000486"/>
     </inertial>
     <collision name="link_left_wheel_collision">
-      <origin rpy="0 1.5707 1.5707" xyz="0 0 0"/>
-      <geometry>
-        <cylinder length="0.04" radius="0.1"/>
+      <origin rpy="0 1.570796 1.570796" xyz="0 0 0"/>
+      <geometry>
+        <cylinder length="0.03" radius="0.09"/>
       </geometry>
     </collision>
     <visual name="link_left_wheel_visual">
-      <origin rpy="0 1.5707 1.5707" xyz="0 0 0"/>
-      <geometry>
-        <cylinder length="0.04" radius="0.1"/>
+      <origin rpy="0 0 1.570796" xyz="0 0 0"/>
+      <geometry>
+        <mesh filename="package://maze_generator/urdf/meshes/umouse_wheel.stl" scale="0.003 0.003 0.003"/>
       </geometry>
     </visual>
   </link>
   <joint name="joint_left_wheel" type="continuous">
-    <origin rpy="0 0 0" xyz="-0.05 -0.15 0"/>
+    <origin rpy="0 0 0" xyz="0 -0.231 0.0345"/>
     <child link="link_left_wheel"/>
-    <parent link="link_chassis"/>
+    <parent link="chassis_base"/>
     <axis rpy="0 0 0" xyz="0 1 0"/>
     <limit effort="10000" velocity="1000"/>
@@ -150,5 +222,5 @@
   <link name="imu_link"/>
   <joint name="imu_joint" type="fixed">
-    <parent link="link_chassis"/>
+    <parent link="chassis_base"/>
     <child link="imu_link"/>
     <origin xyz="0 0 0" rpy="0 0 0"/>
@@ -191,22 +263,9 @@
   <!-- LiDAR Sensor -->
   <joint name="scan_joint" type="fixed">
-    <parent link="link_chassis"/>
+    <parent link="chassis_base"/>
     <child link="link_scan"/>
-    <origin xyz="0.15 0 0.06" rpy="0 0 -1.57079"/>
+    <origin xyz="0.20 0 0.324" rpy="0 0 -1.57079"/>
   </joint>
   <link name="link_scan">
-    <visual>
-      <origin xyz="0 0 0" rpy="0 0 0"/>
-      <geometry>
-        <box size="0.05 0.05 0.05"/>
-      </geometry>
-      <material name="black"/>
-    </visual>
-    <collision>
-      <origin xyz="0 0 0" rpy="0 0 0"/>
-      <geometry>
-        <box size="0.05 0.05 0.05"/>
-      </geometry>
-    </collision>
   </link>
   <gazebo reference="link_scan">
@@ -250,5 +309,5 @@
       <odometrySource>world</odometrySource>
       <publishOdomTF>true</publishOdomTF>
-      <robotBaseFrame>link_chassis</robotBaseFrame>
+      <robotBaseFrame>chassis_base</robotBaseFrame>
       <publishWheelTF>false</publishWheelTF>
       <publishTf>true</publishTf>
@@ -258,8 +317,8 @@
       <leftJoint>joint_left_wheel</leftJoint>
       <rightJoint>joint_right_wheel</rightJoint>
-      <wheelSeparation>0.03</wheelSeparation>
-      <wheelDiameter>0.02</wheelDiameter>
+      <wheelSeparation>0.4635</wheelSeparation>
+      <wheelDiameter>0.18</wheelDiameter>
       <wheelAcceleration>1</wheelAcceleration>
-      <wheelTorque>10</wheelTorque>
+      <wheelTorque>30</wheelTorque>
       <rosDebugLevel>na</rosDebugLevel>
     </plugin>
